Commit message: add setting friction, and make mass larger

File: assets/pure/urdf/pure.urdf (robot description, URDF)
Before this commit: robot pure, 21 links, 20 joints
Links:
- link base_link: mass 1.1584281172172 -> 11.1584281172172

Commit message: optimize scales and gains

File: assets/pure/urdf/pure.urdf (robot description, URDF)
Before this commit: robot pure, 21 links, 20 joints
Links:
- link base_link: mass 11.1584281172172 -> 33.0
